File: 01 KiCad/TheENDGAME x Miao.kicad_sch (KiCad schematic)
At the start: 76 parts, among them J1 Conn_01x01, SW10 SW_Push, SW11 SW_Push, SW12 SW_Push, SW13 SW_Push, SW14 SW_Push, SW15 SW_Push, SW16 SW_Push, SW17 SW_Push, SW18 SW_Push, SW19 SW_Push, SW2 SW_Push, SW20 SW_Push, SW21 SW_Push, SW22 SW_Push, SW23 SW_Push, SW24 SW_Push, SW25 SW_Push, SW26 SW_Push, SW27 SW_Push, SW28 SW_Push, SW29 SW_Push, SW3 SW_Push, SW30 SW_Push, SW31 SW_Push, SW32 SW_Push, SW33 SW_Push, SW34 SW_Push, SW35 SW_Push, SW36 SW_Push, SW37 SW_Push, SW4 SW_Push, SW5 SW_Push, SW6 SW_Push, SW7 SW_Push, SW8 SW_Push, SW9 SW_Push, U1 Miao

Commit message: push prototype pics
Parts:
- D10, D11, D12, D13, D14, D15, D17, D18, D19, D20, D22, D23, D24, D25, D26, D27, D28, D29, D32, D33, D34, D35, D36, D37, D38, D39, D40, D41, D44, D45, D46, D47, D5, D6, D7, D8: footprint UWUmasterGatekeeperHusoLib:Diode_SOD123 triangle clean -> UWUmasterGatekeeperHusoLib:Diode_SOD123 filets triangle
- RSW1, RSW2: footprint UWUmasterGatekeeperHusoLib:SW_SPST_TL3342 ohne Silk -> UWUmasterGatekeeperHusoLib:4X4X1.6mm tact switch Filets
- SW10, SW11, SW12, SW13, SW14, SW15, SW16, SW17, SW18, SW2, SW20, SW21, SW22, SW24, SW25, SW26, SW27, SW28, SW29, SW3, SW30, SW31, SW32, SW33, SW34, SW35, SW36, SW4, SW6, SW7, SW8, SW9: footprint UWUmasterGatekeeperHusoLib:SW_choc_v1_HS_1u_eblaster_purp_MBK_blk -> UWUmasterGatekeeperHusoLib:SW_choc_v1_HS_1u_filets_MBK_blk
- SW19, SW23, SW37, SW5: footprint UWUmasterGatekeeperHusoLib:SW_choc_v1_HS_1_5u_eblaster_purp_MBK_blk -> UWUmasterGatekeeperHusoLib:SW_choc_v1_HS_1_5u_filets_MBK_blk

Commit message: fixed brainfart with mcu pinout
Parts:
- U1: footprint UWUmasterGatekeeperHusoLib:Miao_17_18_short_CUTOUT_MCU_FACING_UP -> UWUmasterGatekeeperHusoLib:Miao_THT_plus_SMD_17_18_short_THT_CUTOUT_MCU_FACING_UP fixxxed
Connections:
- net boot: now also RSW2.2; no longer RSW1.2
- net col0: now also U1.18 (P3.3); no longer U1.17 (P1.0)
- net col1: now also U1.1 (P3.2); no longer U1.11 (P1.5)
- net col2: now also U1.2 (P1.1); no longer U1.10 (P1.6)
- net col3: now also U1.3 (P1.2); no longer U1.9 (P1.7)
- net col4: now also U1.7 (P3.1); no longer U1.8 (RX/CS)
- net col5: now also U1.8 (RX/CS); no longer U1.4 (P1.3)
- net col6: now also U1.9 (P1.7); no longer U1.3 (P1.2)
- net col7: now also U1.10 (P1.6); no longer U1.2 (P1.1)
- net col8: now also U1.11 (P1.5); no longer U1.1 (P3.2)
- net col9: now also U1.17 (P1.0); no longer U1.18 (P3.3)
- net reset: now also RSW1.2; no longer RSW2.2
- net row1: now also U1.6 (P3.4); no longer U1.7 (P3.1)
- net row2: now also U1.5 (P3.5); no longer U1.6 (P3.4)
- net row3: now also U1.4 (P1.3); no longer U1.5 (P3.5)
Changed lines of the file:
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@@
     (stroke (width 0) (type default))
   )
-  (text "Reset" (at 134.62 180.34 0)
+  (text "Reset" (at 109.22 179.07 0)
     (effects (font (size 2.9972 2.9972)) (justify left bottom))
   )
-  (text "Boot" (at 110.49 180.34 0)
+  (text "Boot" (at 135.89 179.07 0)
     (effects (font (size 2.9972 2.9972)) (justify left bottom))
   )
-  (global_label "row3" (shape input) (at 33.02 40.64 180) (fields_autoplaced)
+  (global_label "row3" (shape input) (at 33.02 38.1 180) (fields_autoplaced)
     (effects (font (size 1.27 1.27)) (justify right))
-    (property "Intersheetrefs" "${INTERSHEET_REFS}" (at 25.5596 40.64 0)
+    (property "Intersheetrefs" "${INTERSHEET_REFS}" (at 25.5596 38.1 0)
       (effects (font (size 1.27 1.27)) (justify right) hide)
     )
   )
-  (global_label "col0" (shape input) (at 55.88 26.67 0) (fields_autoplaced)
+  (global_label "col0" (shape input) (at 33.02 26.67 180) (fields_autoplaced)
+    (effects (font (size 1.27 1.27)) (justify right))
+    (property "Intersheetrefs" "${INTERSHEET_REFS}" (at 25.9225 26.67 0)
+      (effects (font (size 1.27 1.27)) (justify right) hide)
+    )
+  )
+  (global_label "col9" (shape input) (at 55.88 26.67 0) (fields_autoplaced)
     (effects (font (size 1.27 1.27)) (justify left))
     (property "Intersheetrefs" "${INTERSHEET_REFS}" (at 62.9775 26.67 0)
@@
     )
   )
-  (global_label "col9" (shape input) (at 33.02 26.67 180) (fields_autoplaced)
-    (effects (font (size 1.27 1.27)) (justify right))
-    (property "Intersheetrefs" "${INTERSHEET_REFS}" (at 25.9225 26.67 0)
-      (effects (font (size 1.27 1.27)) (justify right) hide)
-    )
-  )
   (global_label "gnd" (shape input) (at 110.49 191.77 180) (fields_autoplaced)
     (effects (font (size 1.27 1.27)) (justify right))
@@
     )
   )
-  (global_label "col3" (shape input) (at 55.88 43.18 0) (fields_autoplaced)
-    (effects (font (size 1.27 1.27)) (justify left))
-    (property "Intersheetrefs" "${INTERSHEET_REFS}" (at 62.9775 43.18 0)
-      (effects (font (size 1.27 1.27)) (justify left) hide)
+  (global_label "col3" (shape input) (at 33.02 35.56 180) (fields_autoplaced)
+    (effects (font (size 1.27 1.27)) (justify right))
+    (property "Intersheetrefs" "${INTERSHEET_REFS}" (at 25.9225 35.56 0)
+      (effects (font (size 1.27 1.27)) (justify right) hide)
     )
   )
@@
     )
   )
-  (global_label "col1" (shape input) (at 55.88 38.1 0) (fields_autoplaced)
-    (effects (font (size 1.27 1.27)) (justify left))
-    (property "Intersheetrefs" "${INTERSHEET_REFS}" (at 62.9775 38.1 0)
-      (effects (font (size 1.27 1.27)) (justify left) hide)
+  (global_label "col1" (shape input) (at 33.02 30.48 180) (fields_autoplaced)
+    (effects (font (size 1.27 1.27)) (justify right))
+    (property "Intersheetrefs" "${INTERSHEET_REFS}" (at 25.9225 30.48 0)
+      (effects (font (size 1.27 1.27)) (justify right) hide)
     )
   )
@@
     )
   )
-  (global_label "col5" (shape input) (at 33.02 38.1 180) (fields_autoplaced)
-    (effects (font (size 1.27 1.27)) (justify right))
-    (property "Intersheetrefs" "${INTERSHEET_REFS}" (at 25.9225 38.1 0)
-      (effects (font (size 1.27 1.27)) (justify right) hide)
-    )
-  )
-  (global_label "col6" (shape input) (at 33.02 35.56 180) (fields_autoplaced)
-    (effects (font (size 1.27 1.27)) (justify right))
-    (property "Intersheetrefs" "${INTERSHEET_REFS}" (at 25.9225 35.56 0)
-      (effects (font (size 1.27 1.27)) (justify right) hide)
-    )
-  )
-  (global_label "boot" (shape input) (at 120.65 191.77 0) (fields_autoplaced)
+  (global_label "col5" (shape input) (at 55.88 45.72 0) (fields_autoplaced)
     (effects (font (size 1.27 1.27)) (justify left))
-    (property "Intersheetrefs" "${INTERSHEET_REFS}" (at 127.8079 191.77 0)
+    (property "Intersheetrefs" "${INTERSHEET_REFS}" (at 62.9775 45.72 0)
+      (effects (font (size 1.27 1.27)) (justify left) hide)
+    )
+  )
+  (global_label "col6" (shape input) (at 55.88 43.18 0) (fields_autoplaced)
+    (effects (font (size 1.27 1.27)) (justify left))
+    (property "Intersheetrefs" "${INTERSHEET_REFS}" (at 62.9775 43.18 0)
+      (effects (font (size 1.27 1.27)) (justify left) hide)
+    )
+  )
+  (global_label "boot" (shape input) (at 146.05 191.77 0) (fields_autoplaced)
+    (effects (font (size 1.27 1.27)) (justify left))
+    (property "Intersheetrefs" "${INTERSHEET_REFS}" (at 153.2079 191.77 0)
       (effects (font (size 1.27 1.27)) (justify left) hide)
     )
@@
     )
   )
-  (global_label "col8" (shape input) (at 33.02 30.48 180) (fields_autoplaced)
+  (global_label "col8" (shape input) (at 55.88 38.1 0) (fields_autoplaced)
+    (effects (font (size 1.27 1.27)) (justify left))
+    (property "Intersheetrefs" "${INTERSHEET_REFS}" (at 62.9775 38.1 0)
+      (effects (font (size 1.27 1.27)) (justify left) hide)
+    )
+  )
+  (global_label "col2" (shape input) (at 33.02 33.02 180) (fields_autoplaced)
     (effects (font (size 1.27 1.27)) (justify right))
-    (property "Intersheetrefs" "${INTERSHEET_REFS}" (at 25.9225 30.48 0)
+    (property "Intersheetrefs" "${INTERSHEET_REFS}" (at 25.9225 33.02 0)
       (effects (font (size 1.27 1.27)) (justify right) hide)
     )
   )
-  (global_label "col2" (shape input) (at 55.88 40.64 0) (fields_autoplaced)
+  (global_label "col4" (shape input) (at 33.02 45.72 180) (fields_autoplaced)
+    (effects (font (size 1.27 1.27)) (justify right))
+    (property "Intersheetrefs" "${INTERSHEET_REFS}" (at 25.9225 45.72 0)
+      (effects (font (size 1.27 1.27)) (justify right) hide)
+    )
+  )
+  (global_label "reset" (shape input) (at 120.65 191.77 0) (fields_autoplaced)
     (effects (font (size 1.27 1.27)) (justify left))
-    (property "Intersheetrefs" "${INTERSHEET_REFS}" (at 62.9775 40.64 0)
-      (effects (font (size 1.27 1.27)) (justify left) hide)
-    )
-  )
-  (global_label "col4" (shape input) (at 55.88 45.72 0) (fields_autoplaced)
-    (effects (font (size 1.27 1.27)) (justify left))
-    (property "Intersheetrefs" "${INTERSHEET_REFS}" (at 62.9775 45.72 0)
-      (effects (font (size 1.27 1.27)) (justify left) hide)
-    )
-  )
-  (global_label "reset" (shape input) (at 146.05 191.77 0) (fields_autoplaced)
-    (effects (font (size 1.27 1.27)) (justify left))
-    (property "Intersheetrefs" "${INTERSHEET_REFS}" (at 19.05 152.4 0)
+    (property "Intersheetrefs" "${INTERSHEET_REFS}" (at -6.35 152.4 0)
       (effects (font (size 1.27 1.27)) hide)
     )
@@
     )
   )
-  (global_label "row2" (shape input) (at 33.02 43.18 180) (fields_autoplaced)
+  (global_label "row2" (shape input) (at 33.02 40.64 180) (fields_autoplaced)
     (effects (font (size 1.27 1.27)) (justify right))
-    (property "Intersheetrefs" "${INTERSHEET_REFS}" (at 25.5596 43.18 0)
+    (property "Intersheetrefs" "${INTERSHEET_REFS}" (at 25.5596 40.64 0)
       (effects (font (size 1.27 1.27)) (justify right) hide)
     )
@@
     )
   )
-  (global_label "col7" (shape input) (at 33.02 33.02 180) (fields_autoplaced)
+  (global_label "col7" (shape input) (at 55.88 40.64 0) (fields_autoplaced)
+    (effects (font (size 1.27 1.27)) (justify left))
+    (property "Intersheetrefs" "${INTERSHEET_REFS}" (at 62.9775 40.64 0)
+      (effects (font (size 1.27 1.27)) (justify left) hide)
+    )
+  )
+  (global_label "row1" (shape input) (at 33.02 43.18 180) (fields_autoplaced)
     (effects (font (size 1.27 1.27)) (justify right))
-    (property "Intersheetrefs" "${INTERSHEET_REFS}" (at 25.9225 33.02 0)
-      (effects (font (size 1.27 1.27)) (justify right) hide)
-    )
-  )
-  (global_label "row1" (shape input) (at 33.02 45.72 180) (fields_autoplaced)
-    (effects (font (size 1.27 1.27)) (justify right))
-    (property "Intersheetrefs" "${INTERSHEET_REFS}" (at 25.5596 45.72 0)
+    (property "Intersheetrefs" "${INTERSHEET_REFS}" (at 25.5596 43.18 0)
       (effects (font (size 1.27 1.27)) (justify right) hide)
     )
@@
       (effects (font (size 1.27 1.27)))
     )
-    (property "Footprint" "UWUmasterGatekeeperHusoLib:Miao_17_18_short_CUTOUT_MCU_FACING_UP" (at 48.26 41.91 0)
-      (effects (font (size 1.27 1.27)) hide)
-    )
+    (property "Footprint" "UWUmasterGatekeeperHusoLib:Miao_THT_plus_SMD_17_18_short_THT_CUTOUT_MCU_FACING_UP fixxxed" (at 48.26 41.91 0)
+      (effects (font (size 1.27 1.27)) hide)
+    )
